Commit message: fix(arena_robots): align robot configs for Jazzy Isaac evals
Update robot frames, scan topics, USD dependencies, and Jazzy-compatible robot assets so Ai2_Bot2 and baseline robots resolve consistently in the Isaac evaluation stack.

File: arena_robots/robots/turtlebot/urdf/turtlebot.urdf.xacro (robot description, xacro)
@@ -35,4 +35,7 @@
   <xacro:property name="oakd_pro_y_offset"             value="${0*cm2m}"/>
   <xacro:property name="oakd_pro_z_offset"             value="${9.676*cm2m}"/>
+  <xacro:property name="top_down_camera_x_offset"      value="${0*cm2m}"/>
+  <xacro:property name="top_down_camera_y_offset"      value="${0*cm2m}"/>
+  <xacro:property name="top_down_camera_z_offset"      value="${105*cm2m}"/>
   <!-- Shell Link -->
   <joint name="shell_link_joint" type="fixed">
@@ -104,4 +107,37 @@
     <origin xyz="${oakd_pro_x_offset} ${oakd_pro_y_offset} ${oakd_pro_z_offset}"/>
   </xacro:oakd>
+  <joint name="top_down_camera_joint" type="fixed">
+    <parent link="shell_link"/>
+    <child link="top_down_camera_frame"/>
+    <origin xyz="${top_down_camera_x_offset} ${top_down_camera_y_offset} ${top_down_camera_z_offset}" rpy="0 ${-pi/2} 0"/>
+  </joint>
+  <link name="top_down_camera_frame" />
+  <joint name="top_down_camera_optical_joint" type="fixed">
+    <parent link="top_down_camera_frame"/>
+    <child link="top_down_camera_optical_frame"/>
+    <origin xyz="0 0 0" rpy="${-pi/2} 0 ${-pi/2}"/>
+  </joint>
+  <link name="top_down_camera_optical_frame" />
+  <gazebo reference="top_down_camera_frame">
+    <sensor name="top_down_camera" type="camera">
+      <gz_frame_id>$(arg name)/top_down_camera_optical_frame</gz_frame_id>
+      <camera>
+        <horizontal_fov>2.2</horizontal_fov>
+        <image>
+          <width>640</width>
+          <height>640</height>
+          <format>R8G8B8</format>
+        </image>
+        <clip>
+          <near>0.05</near>
+          <far>25.0</far>
+        </clip>
+        <optical_frame_id>$(arg name)/top_down_camera_optical_frame</optical_frame_id>
+      </camera>
+      <always_on>1</always_on>
+      <update_rate>20</update_rate>
+      <visualize>false</visualize>
+    </sensor>
+  </gazebo>
   <!-- Gazebo Sim Plugins -->
   <gazebo>
@@ -167,3 +203,9 @@
   <gazebo reference="side_left_ir_link"></gazebo>
   <gazebo reference="ir_omni_link"></gazebo>
+  <gazebo reference="top_down_camera_joint">
+    <preserveFixedJoint>true</preserveFixedJoint>
+  </gazebo>
+  <gazebo reference="top_down_camera_optical_joint">
+    <preserveFixedJoint>true</preserveFixedJoint>
+  </gazebo>
 </robot>
